File: JLCFiles/Spectra6PCB_83.brd (EAGLE design)
At the start: 92.1 x 33 mm, 95 parts, among them J5 NC, P1 FH12-50S-0.5SH, Q1 310mA/60V/1.6Ω, Q2 20V/4.2A/52mΩ/1.4W, Q3 DMG3415U, U1 GENERIC-SOIC8MSGEQ7N-FILTER, U2 AP2112, U3 ESP-WROOM-3232D-NARROW, U4 MP6211 3.3V

Commit message: PCB_100units
Parts:
- removed JP1: (no value), pinhead:1X04
- added JP6, JP7: JUMPER-SMT_3_1-NC_TRACE_SILK, SparkFun-Jumpers:SMT-JUMPER_3_1-NC_TRACE_SILK
- added SV3: (no value), con-lsta:FE05-1
- added U$5: (no value), SparkFun-Aesthetics:ROHS_LOGO_0.18_IN
- added U$7: (no value), SparkFun-Aesthetics:NO_PB_LOGO_0.120
- added U$8: (no value), logo:ESD_10.00
- moved S3 0.60 mm to (39.9, 17.6)
- turned JP4 to 180 degrees
Connections:
- removed net 3V3: L3.1, L4.1, SV1.1, SV2.1
- removed net N$27: C23.1, R10.2
- new net TN: J4.1, J5.1, JP7.2
- new net TP: J4.2, J5.2, JP6.2
- net !RESET!: now also SV3.1; no longer JP1.1
- net 3.3V: now also L3.1, L4.1, SV1.1, SV2.1
- net BAT: now also JP6.1, JP7.3; no longer J4.2, J5.2
- net BOOT: now also SV3.5; no longer JP1.4
- net GND: now also JP6.3, JP7.1, SV3.4; no longer J4.1, J5.1
- net IC2: now also JP4.3; no longer JP4.1
- net N$35: now also JP4.1; no longer JP4.3
- net RX0: now also SV3.3; no longer JP1.3
- net TX0: now also SV3.2; no longer JP1.2
- net VB: now also C23.1, R10.2
Routing:
- net 3.3V: track 55.7 -> 120.8 mm, vias 3 -> 4
- net 3V3: track 44.8 -> 0.00 mm
- net VB: track 3.89 -> 28.5 mm
- net TP: track 0.00 -> 15.6 mm, vias 0 -> 1
- net TN: track 0.00 -> 12.2 mm, vias 0 -> 1
- net BAT: track 71.8 -> 78.8 mm
- net N$27: track 4.95 -> 0.00 mm, vias 0 -> 1
- net BOOT: track 9.69 -> 7.41 mm
- net GND: vias 8 -> 9
Other:
- board text added: "1"
- board text added: "2"
- board text added: "HW1.2.0"
- board text added: "ID: __________________"
- board text removed: "HW1.0.1"
- board text removed: "Inventors"
