File: JLCFiles/Spectra6PCB_83.sch (EAGLE design)
At the start: 95 parts, among them J5 NC, P1 FH12-50S-0.5SH, Q1 310mA/60V/1.6Ω, Q2 20V/4.2A/52mΩ/1.4W, Q3 DMG3415U, U1 GENERIC-SOIC8MSGEQ7N-FILTER, U2 AP2112, U3 ESP-WROOM-3232D-NARROW, U4 MP6211 3.3V

Commit message: PCB_100units
Parts:
- removed JP1: (no value), pinhead:PINHD-1X4
- added JP6, JP7: JUMPER-SMT_3_1-NC_TRACE_SILK, SparkFun-Jumpers:JUMPER-SMT_3_1-NC_TRACE_SILK
- added SV3: (no value), con-lsta:FE05-1
Connections:
- removed net 3V3: L3.1, L4.1, SV1.1, SV2.1
- removed net N$27: C23.1, R10.2
- new net TN: J4.-, J5.-, JP7.2
- new net TP: J4.+, J5.+, JP6.2
- net !RESET!: now also SV3.1; no longer JP1.1
- net 3.3V: now also L3.1, L4.1, SV1.1, SV2.1
- net BAT: now also JP6.1, JP7.3; no longer J4.+, J5.+
- net BOOT: now also SV3.5; no longer JP1.4
- net GND: now also JP6.3, JP7.1, SV3.4; no longer J4.-, J5.-
- net IC2: now also JP4.3; no longer JP4.1
- net N$35: now also JP4.1; no longer JP4.3
- net RX0: now also SV3.3; no longer JP1.3
- net TX0: now also SV3.2; no longer JP1.2
- net VB: now also C23.1, R10.2
Other:
- moved on the sheet: J1, JP3, JP4, JP5
