File: JLCFiles/Spectra6PCB_93.brd (EAGLE design)
At the start: 92.1 x 33 mm, 100 parts, among them J5 NC, P1 FH12-50S-0.5SH, Q1 310mA/60V/1.6Ω, Q2 20V/4.2A/52mΩ/1.4W, Q3 DMG3415U, U1 GENERIC-SOIC8MSGEQ7N-FILTER, U2 AP2112, U3 ESP-WROOM-3232D-NARROW, U4 MP6211 3.3V

Commit message: JLCPCB
Parts:
- U$4: device USBC6PIN4:USBC6PIN -> USBC6PIN2:USBC6PIN
- moved U$4 4.88 mm to (10.7, 21.8)
Connections:
- net SHLD: now also U$4.P$11, U$4.P$5
Routing:
- net BAT: track 78.8 -> 76.2 mm
- net TP: track 15.6 -> 14.9 mm
Other:
- board size 92.1 x 33 mm -> 92.2 x 33 mm
- board text added: "Boot"
- board text added: "HW1.3.0"
- board text added: "Reset"
- board text removed: "HW1.2.0"
